Commit message: Update RR_planar_robot with realistic MOI values

File: RR_planar_robot.urdf (robot description, URDF)
Before this commit: robot physics, 3 links, 2 joints
Joints:
- joint link1_to_link2: type fixed -> continuous

Commit message: Add end-effector link
For ground truth cartesian data

File: RR_planar_robot.urdf (robot description, URDF)
Before this commit: robot physics, 3 links, 2 joints
Links:
- added link ee, mass 0.1; collision box size=0.06 0.06 0.06; visual box size=0.06 0.06 0.06
- link link1: mass 0.1 -> 1
- link link2: mass 0.1 -> 1
Joints:
- added joint link2_to_ee: type fixed, parent link2, child ee, origin xyz=1.0 0.0 0.0 rpy=0.0 0.0 0.0, axis 0 0 1

Commit message: Update robot
Remove collision
Move starting position to [0,1]

File: RR_planar_robot.urdf (robot description, URDF)
Before this commit: robot physics, 4 links, 3 joints
Links:
- link ee: geometry collision box size=0 0 0; visual box size=0.06 0.06 0.06
- link link1: geometry collision box size=0 0 0; visual box size=1.0 0.05 0.05
- link link2: geometry collision box size=0 0 0; visual box size=1.0 0.05 0.05

Commit message: Add third link

File: RR_planar_robot.urdf (robot description, URDF)
Before this commit: robot physics, 4 links, 3 joints
Links:
- link ee: mass 0.1 -> 0.5; geometry collision box size=0 0 0; visual box size=0.5 0.025 0.025
Joints:
- joint link2_to_ee: origin xyz=1.0 0.0 0.0 rpy=0.0 0.0 0.0 -> xyz=1.0 0.0 0.0 rpy=0.0 0.0 0.4
